File: 75% keyboard/Keyboard.kicad_pcb (KiCad board)
At the start: 2 copper layers, 314.3 x 128.6 mm, 166 parts, among them SW1 RotaryEncoder, U1 nice_nano

Commit message: kicad files
Parts:
- removed SW1: RotaryEncoder, Rotary Encoder:Bourns-PEC11R-4220F-S0024-0-0-0
- added J1: AudioJack4, Connector_Audio:Jack_3.5mm_PJ320D_Horizontal, B.Cu at (384.7, 71.6)
Connections:
- U1 pad 1: A -> T
- U1 pad 2: B -> R1
- U1 pad 21: unconnected-(U1-VCC-Pad21) -> R2
- U1 pad 3: C -> S
Routing:
- net R2: track 0.00 -> 287.2 mm, vias 0 -> 3
- net B: track 275.6 -> 0.00 mm, vias 2 -> 0
- net C: track 275.0 -> 0.00 mm
- net S: track 0.00 -> 273.2 mm
- net A: track 269.8 -> 0.00 mm
- net T: track 0.00 -> 264.8 mm
- net R1: track 0.00 -> 264.0 mm, vias 0 -> 4
Other:
- board size 314.3 x 128.6 mm -> 314.3 x 133.4 mm

Commit message: kicad + CAD files
CAD was created using Autodesk Inventor
Parts:
- moved J1 3.18 mm to (381.5, 71.6)
Routing:
- net T: track 264.8 -> 261.6 mm
- net S: track 273.2 -> 270.0 mm
- net R2: track 287.2 -> 284.0 mm
- net R1: track 264.0 -> 263.0 mm
Changed lines of the file:
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@@
 	(footprint "Connector_Audio:Jack_3.5mm_PJ320D_Horizontal"
 		(layer "B.Cu")
-		(at 384.65125 71.59375 -90)
+		(at 381.47625 71.59375 -90)
 		(descr "Headphones with microphone connector, 3.5mm, 4 pins (http://www.qingpu-electronics.com/en/products/WQP-PJ320D-72.html)")
 		(tags "3.5mm jack mic microphone phones headphones 4pins audio plug")
@@
 	)
 	(segment
-		(start 376.71375 69.85)
-		(end 378.145 68.41875)
-		(width 0.2)
-		(layer "B.Cu")
-		(net 102)
-	)
-	(segment
 		(start 125.095 72.23125)
 		(end 121.6715 75.65475)
@@
 	)
 	(segment
-		(start 378.145 68.41875)
-		(end 381.40125 68.41875)
+		(start 364.8075 71.4375)
+		(end 125.095 71.4375)
 		(width 0.2)
 		(layer "B.Cu")
@@
 	)
 	(segment
-		(start 364.8075 71.4375)
-		(end 125.095 71.4375)
+		(start 108.1295 85.725)
+		(end 107.6325 85.725)
 		(width 0.2)
 		(layer "B.Cu")
@@
 	)
 	(segment
-		(start 108.1295 85.725)
-		(end 107.6325 85.725)
+		(start 376.71375 69.85)
+		(end 378.145 68.41875)
 		(width 0.2)
 		(layer "B.Cu")
@@
 	)
 	(segment
-		(start 374.245 68.2625)
-		(end 381.40125 75.41875)
+		(start 378.145 68.41875)
+		(end 378.22625 68.41875)
 		(width 0.2)
 		(layer "B.Cu")
-		(net 103)
+		(net 102)
 	)
 	(segment
@@
 	)
 	(segment
+		(start 367.9825 68.2625)
+		(end 375.13875 75.41875)
+		(width 0.2)
+		(layer "B.Cu")
+		(net 103)
+	)
+	(segment
+		(start 375.13875 75.41875)
+		(end 378.22625 75.41875)
+		(width 0.2)
+		(layer "B.Cu")
+		(net 103)
+	)
+	(segment
 		(start 121.12625 68.2625)
-		(end 374.245 68.2625)
+		(end 367.9825 68.2625)
 		(width 0.2)
 		(layer "B.Cu")
@@
 	)
 	(segment
-		(start 375.27313 76.51875)
-		(end 387.90125 76.51875)
+		(start 125.4125 69.05625)
+		(end 367.81063 69.05625)
 		(width 0.2)
 		(layer "B.Cu")
@@
 	)
 	(segment
-		(start 120.015 74.45375)
-		(end 125.4125 69.05625)
+		(start 375.27313 76.51875)
+		(end 384.72625 76.51875)
 		(width 0.2)
 		(layer "B.Cu")
@@
 	)
 	(segment
-		(start 125.4125 69.05625)
-		(end 367.81063 69.05625)
+		(start 120.015 74.45375)
+		(end 125.4125 69.05625)
 		(width 0.2)
 		(layer "B.Cu")
@@
 	)
 	(segment
-		(start 364.8075 69.85)
-		(end 367.18875 69.85)
+		(start 379.095 70.55)
+		(end 378.22625 71.41875)
 		(width 0.2)
 		(layer "B.Cu")
@@
 	)
 	(segment
-		(start 379.8325 69.85)
-		(end 381.40125 71.41875)
+		(start 379.095 69.85)
+		(end 379.095 70.55)
 		(width 0.2)
 		(layer "B.Cu")
@@
 	)
 	(segment
-		(start 379.095 69.85)
-		(end 379.8325 69.85)
+		(start 364.8075 69.85)
+		(end 367.18875 69.85)
 		(width 0.2)
 		(layer "B.Cu")
