File: macropad/practice.kicad_pcb (KiCad board)
At the start: 2 copper layers, 77.8 x 115.1 mm, 39 parts, among them J1 AudioJack4, U1 ProMicro

Commit message: kicad files
Other:
- board size 77.8 x 115.1 mm -> 85.7 x 121.4 mm
Changed lines of the file:
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@@
 	)
 	(gr_line
-		(start 36.195 24.1275)
-		(end 112.395 24.1275)
-		(stroke
-			(width 0.05)
-			(type default)
-		)
-		(layer "Edge.Cuts")
-	)
-	(gr_arc
-		(start 113.18875 138.4275)
-		(mid 112.956266 138.988766)
-		(end 112.395 139.22125)
+		(start 31.4325 21.74625)
+		(end 117.1575 21.74625)
 		(stroke
 			(width 0.05)
@@
 	)
 	(gr_line
-		(start 35.40125 43.1775)
-		(end 35.40125 24.92125)
+		(start 31.4325 21.74625)
+		(end 31.4325 143.19)
 		(stroke
 			(width 0.05)
@@
 	)
 	(gr_line
-		(start 35.40125 43.1775)
-		(end 35.40125 138.4275)
+		(start 117.1575 143.19)
+		(end 31.4325 143.19)
 		(stroke
 			(width 0.05)
@@
 	)
 	(gr_line
-		(start 112.395 139.22125)
-		(end 36.195 139.22125)
+		(start 117.1575 143.19)
+		(end 117.1575 21.74625)
 		(stroke
 			(width 0.05)
-			(type default)
-		)
-		(layer "Edge.Cuts")
-	)
-	(gr_arc
-		(start 112.395 24.1275)
-		(mid 112.956266 24.359984)
-		(end 113.18875 24.92125)
-		(stroke
-			(width 0.05)
-			(type default)
-		)
-		(layer "Edge.Cuts")
-	)
-	(gr_line
-		(start 113.18875 24.92125)
-		(end 113.18875 42.38375)
-		(stroke
-			(width 0.05)
-			(type default)
-		)
-		(layer "Edge.Cuts")
-	)
-	(gr_line
-		(start 113.18875 138.4275)
-		(end 113.18875 42.38375)
-		(stroke
-			(width 0.05)
-			(type default)
-		)
-		(layer "Edge.Cuts")
-	)
-	(gr_arc
-		(start 36.195 139.22125)
-		(mid 35.633734 138.988766)
-		(end 35.40125 138.4275)
-		(stroke
-			(width 0.05)
-			(type default)
-		)
-		(layer "Edge.Cuts")
-	)
-	(gr_arc
-		(start 35.40125 24.92125)
-		(mid 35.633734 24.359984)
-		(end 36.195 24.1275)
-		(stroke
-			(width 0.05)
